Commit message: Add Isaac Sim model, datasheet limits and verified gripper geometry

File: src/lwa4p_description/urdf/lwa4p.urdf.xacro (robot description, xacro)
@@ -4,8 +4,11 @@
 <robot name="lwa4p" xmlns:xacro="http://www.ros.org/wiki/xacro">
   <xacro:property name="mesh" value="package://lwa4p_description/meshes/lwa4p"/>
+  <!-- limits from the SCHUNK datasheets: range = preset software limit switches
+       (LWA 4P manual 3.2: +-170 deg, axis 3 +-155 deg) minus a small margin,
+       72 deg/s, effort = max. torque (ERB 145: 64 Nm, ERB 115: 19 Nm) -->
   <xacro:property name="safety_offset" value="0.02"/>
-  <xacro:property name="lim" value="${2.967 - safety_offset}"/>
-  <xacro:property name="lim3" value="${2.714 - safety_offset}"/>
-  <xacro:property name="vel" value="1.26"/>
+  <xacro:property name="lim" value="${radians(170) - safety_offset}"/>
+  <xacro:property name="lim3" value="${radians(155) - safety_offset}"/>
+  <xacro:property name="vel" value="${radians(72)}"/>
   <material name="schunk_blue"><color rgba="0.0 0.25 0.6 1.0"/></material>
   <material name="schunk_grey"><color rgba="0.75 0.75 0.75 1.0"/></material>
@@ -69,20 +72,20 @@
   </link>
   <xacro:arm_joint n="1" parent="arm_base_link" child="arm_1_link"
-                   xyz="0 0 0" rpy="0 0 0" effort="370" lower="${-lim}" upper="${lim}"/>
+                   xyz="0 0 0" rpy="0 0 0" effort="64" lower="${-lim}" upper="${lim}"/>
   <xacro:arm_link name="arm_1_link" stl="arm_1_link" material="schunk_blue"/>
   <xacro:arm_joint n="2" parent="arm_1_link" child="arm_2_link"
-                   xyz="0 0 0" rpy="1.5708 0 0" effort="370" lower="${-lim}" upper="${lim}"/>
+                   xyz="0 0 0" rpy="1.5708 0 0" effort="64" lower="${-lim}" upper="${lim}"/>
   <xacro:arm_link name="arm_2_link" stl="arm_2_link" material="schunk_grey"/>
   <xacro:arm_joint n="3" parent="arm_2_link" child="arm_3_link"
-                   xyz="0 0.350 0" rpy="0 3.14159 0" effort="176" lower="${-lim3}" upper="${lim3}"/>
+                   xyz="0 0.350 0" rpy="0 3.14159 0" effort="64" lower="${-lim3}" upper="${lim3}"/>
   <xacro:arm_link name="arm_3_link" stl="arm_3_link" material="schunk_blue"/>
   <xacro:arm_joint n="4" parent="arm_3_link" child="arm_4_link"
-                   xyz="0 0 0" rpy="-1.5708 3.14159 0" effort="176" lower="${-lim}" upper="${lim}"/>
+                   xyz="0 0 0" rpy="-1.5708 3.14159 0" effort="64" lower="${-lim}" upper="${lim}"/>
   <xacro:arm_link name="arm_4_link" stl="arm_4_link" material="schunk_grey"/>
   <xacro:arm_joint n="5" parent="arm_4_link" child="arm_5_link"
-                   xyz="0 0.005263 0.305" rpy="1.5708 0 3.14159" effort="41.6" lower="${-lim}" upper="${lim}"/>
+                   xyz="0 0.005263 0.305" rpy="1.5708 0 3.14159" effort="19" lower="${-lim}" upper="${lim}"/>
   <xacro:arm_link name="arm_5_link" stl="arm_5_link" material="schunk_blue"/>
   <xacro:arm_joint n="6" parent="arm_5_link" child="arm_6_link"
-                   xyz="0 0 0" rpy="-1.5708 0 0" effort="20.1" lower="${-lim}" upper="${lim}"/>
+                   xyz="0 0 0" rpy="-1.5708 0 0" effort="19" lower="${-lim}" upper="${lim}"/>
   <xacro:arm_link name="arm_6_link" stl="arm_6_link" material="schunk_grey"/>
   <!-- tool flange face (end of the arm_6 mesh, z = 0.084) -->

File: src/lwa4p_description/urdf/wsg50.urdf.xacro (robot description, xacro)
@@ -1,20 +1,34 @@
 <?xml version="1.0"?>
-<!-- Weiss/Schunk WSG 50-110 on the FWA115 adapter, simple box geometry.
-     Dimensions are approximate (measure and adjust): adapter 20 mm,
-     housing 146 x 52 x 72 mm, fingers 20 x 30 x 90 mm.
+<!-- Weiss/Schunk WSG 50-110 on an adapter plate, simple box geometry.
+     From the WSG 50 manual (05.00, 389474, "3.1 Outer dimensions"):
+       housing 146 x 50 x 72.5 mm (x = jaw direction), Ø50 ISO mounting in the
+       centre of the bottom face, base jaws stick out to 96.5 mm (24 mm above
+       the housing), ~18 mm wide in x, jaw inner faces 0..110 mm apart.
+       Weight 1.15 kg, 5..80 N, 5..420 mm/s.
+     Measured on the real gripper: the mounted fingers reach 9.75 mm further
+       inwards than each jaw (fingertip gap = jaw width - 19.5 mm).
+     NOT measured yet (change when you know them):
+       adapter_h (flange -> housing bottom), jaw_d (jaw depth in y),
+       finger_t / finger_w / finger_l (finger thickness, width, length above
+       the jaw). finger_l is chosen so the fingertips are 162 mm above the
+       housing bottom, as in the earlier model (keeps gripper_tcp unchanged).
      gripper_joint = fingertip GAP in metres (same number the gripper node,
-     MoveIt and `arm_cmd.sh grip` use). Each finger mimics half of it.
-     Inertials are rough guesses (WSG 50 ~1.2 kg), only Gazebo uses them. -->
+     MoveIt and `arm_cmd.sh grip` use). Each finger mimics half of it. -->
 <robot xmlns:xacro="http://www.ros.org/wiki/xacro">
   <xacro:macro name="wsg50" params="parent yaw:=0">
     <xacro:property name="adapter_h" value="0.020"/>
     <xacro:property name="body_x" value="0.146"/>
-    <xacro:property name="body_y" value="0.052"/>
-    <xacro:property name="body_h" value="0.072"/>
+    <xacro:property name="body_y" value="0.050"/>
+    <xacro:property name="body_h" value="0.0725"/>
+    <xacro:property name="jaw_w" value="0.018"/>
+    <xacro:property name="jaw_d" value="0.030"/>
+    <xacro:property name="jaw_h" value="0.024"/>
+    <xacro:property name="jaw_inset" value="0.00975"/>
     <xacro:property name="finger_t" value="0.020"/>
     <xacro:property name="finger_w" value="0.030"/>
-    <xacro:property name="finger_l" value="0.090"/>
+    <xacro:property name="finger_l" value="0.0655"/>
     <xacro:property name="gap_max" value="0.0895"/>
     <material name="wsg_grey"><color rgba="0.6 0.6 0.62 1.0"/></material>
+    <material name="wsg_jaw"><color rgba="0.35 0.35 0.38 1.0"/></material>
     <material name="wsg_black"><color rgba="0.1 0.1 0.1 1.0"/></material>
     <joint name="gripper_adapter_joint" type="fixed">
@@ -26,14 +40,15 @@
       <visual>
         <origin xyz="0 0 ${adapter_h / 2}"/>
-        <geometry><cylinder radius="0.042" length="${adapter_h}"/></geometry>
+        <geometry><cylinder radius="0.0325" length="${adapter_h}"/></geometry>
         <material name="wsg_grey"/>
       </visual>
       <collision>
         <origin xyz="0 0 ${adapter_h / 2}"/>
-        <geometry><cylinder radius="0.042" length="${adapter_h}"/></geometry>
+        <geometry><cylinder radius="0.0325" length="${adapter_h}"/></geometry>
       </collision>
       <inertial>
-        <mass value="0.2"/>
-        <inertia ixx="1e-4" ixy="0" ixz="0" iyy="1e-4" iyz="0" izz="1e-4"/>
+        <origin xyz="0 0 ${adapter_h / 2}"/>
+        <mass value="0.15"/>
+        <inertia ixx="4.5e-5" ixy="0" ixz="0" iyy="4.5e-5" iyz="0" izz="8e-5"/>
       </inertial>
     </link>
@@ -54,6 +69,7 @@
       </collision>
       <inertial>
-        <mass value="1.2"/>
-        <inertia ixx="3e-3" ixy="0" ixz="0" iyy="3e-3" iyz="0" izz="3e-3"/>
+        <origin xyz="0 0 ${body_h / 2}"/>
+        <mass value="0.95"/>
+        <inertia ixx="6.1e-4" ixy="0" ixz="0" iyy="2.1e-3" iyz="0" izz="1.9e-3"/>
       </inertial>
     </link>
@@ -73,4 +89,6 @@
       </inertial>
     </link>
+    <!-- one finger = base jaw (on the housing top) + mounted finger.
+         Link origin: on the housing top, at the inner (gripping) face of the finger. -->
     <xacro:macro name="finger" params="side sign">
       <joint name="gripper_finger_${side}_joint" type="prismatic">
@@ -82,19 +100,27 @@
         <mimic joint="gripper_joint" multiplier="${sign * 0.5}" offset="0"/>
       </joint>
-      <!-- link origin = inner (gripping) face of the finger -->
       <link name="gripper_finger_${side}_link">
         <visual>
-          <origin xyz="${sign * finger_t / 2} 0 ${finger_l / 2}"/>
+          <origin xyz="${sign * (jaw_inset + jaw_w / 2)} 0 ${jaw_h / 2}"/>
+          <geometry><box size="${jaw_w} ${jaw_d} ${jaw_h}"/></geometry>
+          <material name="wsg_jaw"/>
+        </visual>
+        <visual>
+          <origin xyz="${sign * finger_t / 2} 0 ${jaw_h + finger_l / 2}"/>
           <geometry><box size="${finger_t} ${finger_w} ${finger_l}"/></geometry>
           <material name="wsg_black"/>
         </visual>
         <collision>
-          <origin xyz="${sign * finger_t / 2} 0 ${finger_l / 2}"/>
+          <origin xyz="${sign * (jaw_inset + jaw_w / 2)} 0 ${jaw_h / 2}"/>
+          <geometry><box size="${jaw_w} ${jaw_d} ${jaw_h}"/></geometry>
+        </collision>
+        <collision>
+          <origin xyz="${sign * finger_t / 2} 0 ${jaw_h + finger_l / 2}"/>
           <geometry><box size="${finger_t} ${finger_w} ${finger_l}"/></geometry>
         </collision>
         <inertial>
-          <origin xyz="${sign * finger_t / 2} 0 ${finger_l / 2}"/>
-          <mass value="0.05"/>
-          <inertia ixx="4e-5" ixy="0" ixz="0" iyy="4e-5" iyz="0" izz="5e-6"/>
+          <origin xyz="${sign * 0.012} 0 0.035"/>
+          <mass value="0.1"/>
+          <inertia ixx="5e-5" ixy="0" ixz="0" iyy="5.5e-5" iyz="0" izz="1.5e-5"/>
         </inertial>
       </link>
@@ -106,5 +132,5 @@
       <parent link="gripper_body_link"/>
       <child link="gripper_tcp"/>
-      <origin xyz="0 0 ${body_h + finger_l - 0.015}" rpy="0 0 0"/>
+      <origin xyz="0 0 ${body_h + jaw_h + finger_l - 0.015}" rpy="0 0 0"/>
     </joint>
     <link name="gripper_tcp"/>
